Commit message: Updated models

File: robotiq_2f_140_gripper_visualization/urdf/robotiq_arg2f.xacro (robot description, xacro)
@@ -38,3 +38,33 @@
     <xacro:inner_knuckle prefix="${prefix}" fingerprefix="${fingerprefix}" stroke="${stroke}"/>
   </xacro:macro>
+  <xacro:macro name="robotiq_arg2f_gazebo" params="prefix">
+		<gazebo>
+			<!-- loading plugin: mimic joints works in gazebo now-->
+			<plugin filename="libroboticsgroup_gazebo_mimic_joint_plugin.so" name="${prefix}mimic_robotiq_140_4">
+				<joint>${prefix}finger_joint</joint>
+				<mimicJoint>${prefix}right_outer_knuckle_joint</mimicJoint>
+				<multiplier>-1.0</multiplier>
+			</plugin>
+			<plugin filename="libroboticsgroup_gazebo_mimic_joint_plugin.so" name="${prefix}mimic_robotiq_140_2">
+				<joint>${prefix}finger_joint</joint>
+				<mimicJoint>${prefix}left_inner_finger_joint</mimicJoint>
+				<multiplier>1.0</multiplier>
+			</plugin>
+			<plugin filename="libroboticsgroup_gazebo_mimic_joint_plugin.so" name="${prefix}mimic_robotiq_140_1">
+				<joint>${prefix}finger_joint</joint>
+				<mimicJoint>${prefix}right_inner_finger_joint</mimicJoint>
+				<multiplier>1.0</multiplier>
+			</plugin>
+			<plugin filename="libroboticsgroup_gazebo_mimic_joint_plugin.so" name="${prefix}mimic_robotiq_140_3">
+				<joint>${prefix}finger_joint</joint>
+				<mimicJoint>${prefix}left_inner_knuckle_joint</mimicJoint>
+				<multiplier>-1.0</multiplier>
+			</plugin>
+			<plugin filename="libroboticsgroup_gazebo_mimic_joint_plugin.so" name="${prefix}mimic_robotiq_140_5">
+				<joint>${prefix}finger_joint</joint>
+				<mimicJoint>${prefix}right_inner_knuckle_joint</mimicJoint>
+				<multiplier>-1.0</multiplier>
+			</plugin>
+		</gazebo>
+	</xacro:macro>
 </robot>

File: robotiq_2f_140_gripper_visualization/urdf/robotiq_arg2f_140_model_macro.xacro (robot description, xacro)
@@ -210,4 +210,5 @@
     <xacro:right_outer_knuckle_joint prefix="${prefix}"/>
     <xacro:robotiq_arg2f_transmission prefix="${prefix}"/>
+    <xacro:robotiq_arg2f_gazebo prefix="${prefix}" />
   </xacro:macro>
 </robot>

File: robotiq_2f_85_gripper_visualization/urdf/robotiq_arg2f.xacro (robot description, xacro)
@@ -38,3 +38,33 @@
     <xacro:inner_knuckle prefix="${prefix}" fingerprefix="${fingerprefix}" stroke="${stroke}"/>
   </xacro:macro>
+  <xacro:macro name="robotiq_arg2f_gazebo" params="prefix">
+		<gazebo>
+			<!-- loading plugin: mimic joints works in gazebo now-->
+			<plugin filename="libroboticsgroup_gazebo_mimic_joint_plugin.so" name="${prefix}mimic_robotiq_85_4">
+				<joint>${prefix}finger_joint</joint>
+				<mimicJoint>${prefix}right_outer_knuckle_joint</mimicJoint>
+				<multiplier>1.0</multiplier>
+			</plugin>
+			<plugin filename="libroboticsgroup_gazebo_mimic_joint_plugin.so" name="${prefix}mimic_robotiq_85_2">
+				<joint>${prefix}finger_joint</joint>
+				<mimicJoint>${prefix}left_inner_finger_joint</mimicJoint>
+				<multiplier>-1.0</multiplier>
+			</plugin>
+			<plugin filename="libroboticsgroup_gazebo_mimic_joint_plugin.so" name="${prefix}mimic_robotiq_85_1">
+				<joint>${prefix}finger_joint</joint>
+				<mimicJoint>${prefix}right_inner_finger_joint</mimicJoint>
+				<multiplier>-1.0</multiplier>
+			</plugin>
+			<plugin filename="libroboticsgroup_gazebo_mimic_joint_plugin.so" name="${prefix}mimic_robotiq_85_3">
+				<joint>${prefix}finger_joint</joint>
+				<mimicJoint>${prefix}left_inner_knuckle_joint</mimicJoint>
+				<multiplier>1.0</multiplier>
+			</plugin>
+			<plugin filename="libroboticsgroup_gazebo_mimic_joint_plugin.so" name="${prefix}mimic_robotiq_85_5">
+				<joint>${prefix}finger_joint</joint>
+				<mimicJoint>${prefix}right_inner_knuckle_joint</mimicJoint>
+				<multiplier>1.0</multiplier>
+			</plugin>
+		</gazebo>
+	</xacro:macro>
 </robot>

File: robotiq_2f_85_gripper_visualization/urdf/robotiq_arg2f_85_model_macro.xacro (robot description, xacro)
@@ -188,4 +188,5 @@
     <xacro:right_outer_knuckle_joint prefix="${prefix}"/>
     <xacro:robotiq_arg2f_transmission prefix="${prefix}"/>
+    <xacro:robotiq_arg2f_gazebo prefix="${prefix}" />
   </xacro:macro>
 </robot>
